File: ioio-adapter/ioio-adapter.sch (KiCad schematic (older format))
At the start: 19 parts

Commit message: Use INT1 instead of CN interrupt
This will make the interrupt routine faster since there is no
need to check which pin that caused the interrupt and if it was
a positive or negative flank.
Connections:
- net labels added: IOIO_PIN14
- net labels removed: IOIO_PIN18
- wire segments 68 -> 57
Changed lines of the file:
@@
-EESchema Schematic File Version 2  date Sun 09 Jun 2013 09:52:20 PM CEST
+EESchema Schematic File Version 2  date Fri 14 Jun 2013 12:48:07 PM CEST
 LIBS:power
 LIBS:device
@@
 Sheet 1 1
 Title ""
-Date "9 jun 2013"
+Date "14 jun 2013"
 Rev ""
 Comp ""
@@
 Comment4 ""
 $EndDescr
+Wire Wire Line
+	6100 2300 6100 3500
+Wire Wire Line
+	1500 3500 1500 3650
+Wire Wire Line
+	1500 3650 1350 3650
+Wire Wire Line
+	2650 2600 1350 2600
+Wire Wire Line
+	8000 2100 8950 2100
+Wire Wire Line
+	8000 1900 8950 1900
+Wire Wire Line
+	3950 2550 3100 2550
+Wire Wire Line
+	3950 2000 3400 2000
+Wire Wire Line
+	5100 2250 4450 2250
+Connection ~ 6400 1150
+Wire Wire Line
+	6400 1150 4850 1150
+Connection ~ 5900 1150
+Wire Wire Line
+	4850 1700 4850 1800
+Connection ~ 5400 2850
+Wire Wire Line
+	6400 2850 4850 2850
+Wire Wire Line
+	4850 2850 4850 2200
+Wire Wire Line
+	4850 1800 6600 1800
+Connection ~ 6400 2850
+Wire Wire Line
+	5900 2850 5900 2750
+Connection ~ 5900 2300
+Wire Wire Line
+	6400 3250 6400 2400
+Wire Wire Line
+	6400 2400 6600 2400
+Wire Wire Line
+	1300 1150 2150 1150
+Wire Wire Line
+	1350 1550 2150 1550
+Wire Wire Line
+	1350 1050 2150 1050
+Wire Wire Line
+	1500 750  1500 850
+Wire Wire Line
+	1500 850  1350 850
+Wire Wire Line
+	1500 1950 1500 1650
+Wire Wire Line
+	1500 1650 1350 1650
+Wire Wire Line
+	4550 5000 5350 5000
+Wire Wire Line
+	6450 4750 6250 4750
+Wire Wire Line
+	6250 4100 6250 4150
+Wire Wire Line
+	6250 5700 6250 5850
+Wire Wire Line
+	6250 5200 6250 5300
+Wire Wire Line
+	6250 4800 6250 4650
+Wire Wire Line
+	5850 5000 5950 5000
+Connection ~ 6250 4750
+Wire Wire Line
+	5950 5500 5850 5500
+Wire Wire Line
+	4550 5500 5350 5500
+Wire Wire Line
+	1350 1750 1500 1750
+Connection ~ 1500 1750
+Wire Wire Line
+	1350 1250 2150 1250
+Wire Wire Line
+	1350 1350 2150 1350
+Wire Wire Line
+	1350 2700 1500 2700
+Wire Wire Line
+	1500 2700 1500 2900
+Wire Wire Line
+	6400 1050 6400 2100
+Wire Wire Line
+	6400 2100 6600 2100
+Wire Wire Line
+	6600 2300 5900 2300
+Wire Wire Line
+	5900 1150 5900 1200
+Wire Wire Line
+	5400 2000 6600 2000
+Wire Wire Line
+	5400 2450 5400 2850
+Connection ~ 5900 2850
+Wire Wire Line
+	5900 2350 5900 1700
+Wire Wire Line
+	5400 1200 5400 1150
+Wire Wire Line
+	4850 1150 4850 1200
+Wire Wire Line
+	5400 2050 5400 1700
+Connection ~ 5400 2000
+Connection ~ 5400 1150
+Wire Wire Line
+	4550 2000 4450 2000
+Wire Wire Line
+	5600 2550 4450 2550
+Wire Wire Line
+	3950 2250 3100 2250
+Wire Wire Line
+	8950 1800 8000 1800
+Wire Wire Line
+	8000 2000 8950 2000
+Wire Wire Line
+	6100 3500 8950 3500
+Wire Wire Line
+	1350 3850 1500 3850
+Wire Wire Line
+	1500 3850 1500 3950
+Wire Wire Line
+	6950 4750 7550 4750
+Connection ~ 6100 2300
 Text Notes 800  2350 0    60   ~ 0
 Keyboard to control card connector
 Text Notes 550  600  0    60   ~ 0
 Keyboard to keyboard cable connector
-Connection ~ 6100 2000
-Wire Wire Line
-	6100 2000 6100 3500
-Wire Wire Line
-	1500 3500 1500 3650
-Wire Wire Line
-	1500 3650 1350 3650
-Wire Wire Line
-	2650 2600 1350 2600
-Wire Wire Line
-	8000 2100 8950 2100
-Wire Wire Line
-	8000 1900 8950 1900
-Wire Wire Line
-	3950 2550 3100 2550
-Wire Wire Line
-	3950 2000 3400 2000
-Wire Wire Line
-	5100 2250 4450 2250
-Connection ~ 6400 1150
-Wire Wire Line
-	6400 1150 5900 1150
-Wire Wire Line
-	5900 1150 5400 1150
-Wire Wire Line
-	5400 1150 4850 1150
-Connection ~ 5900 1150
-Wire Wire Line
-	4850 1700 4850 1800
-Connection ~ 5400 2850
-Wire Wire Line
-	6400 2850 5900 2850
-Wire Wire Line
-	5900 2850 5400 2850
-Wire Wire Line
-	5400 2850 4850 2850
-Wire Wire Line
-	4850 2850 4850 2200
-Wire Wire Line
-	4850 1800 6600 1800
-Connection ~ 6400 2850
-Wire Wire Line
-	5900 2850 5900 2750
-Connection ~ 5900 2300
-Wire Wire Line
-	6400 3250 6400 2850
-Wire Wire Line
-	6400 2850 6400 2400
-Wire Wire Line
-	6400 2400 6600 2400
-Wire Wire Line
-	1300 1150 2150 1150
-Wire Wire Line
-	1350 1550 2150 1550
-Wire Wire Line
-	1350 1050 2150 1050
-Wire Wire Line
-	1500 750  1500 850
-Wire Wire Line
-	1500 850  1350 850
-Wire Wire Line
-	1500 1950 1500 1750
-Wire Wire Line
-	1500 1750 1500 1650
-Wire Wire Line
-	1500 1650 1350 1650
-Wire Wire Line
-	4550 5000 5350 5000
-Wire Wire Line
-	6450 4750 6250 4750
-Wire Wire Line
-	6250 4100 6250 4150
-Wire Wire Line
-	6250 5700 6250 5850
-Wire Wire Line
-	6250 5200 6250 5300
-Wire Wire Line
-	6250 4650 6250 4750
-Wire Wire Line
-	6250 4750 6250 4800
-Wire Wire Line
-	5850 5000 5950 5000
-Connection ~ 6250 4750
-Wire Wire Line
-	5950 5500 5850 5500
-Wire Wire Line
-	4550 5500 5350 5500
-Wire Wire Line
-	1350 1750 1500 1750
-Connection ~ 1500 1750
-Wire Wire Line
-	1350 1250 2150 1250
-Wire Wire Line
-	1350 1350 2150 1350
-Wire Wire Line
-	1350 2700 1500 2700
-Wire Wire Line
-	1500 2700 1500 2900
-Wire Wire Line
-	6400 1050 6400 1150
-Wire Wire Line
-	6400 1150 6400 2100
-Wire Wire Line
-	6400 2100 6600 2100
-Wire Wire Line
-	6600 2300 5900 2300
-Wire Wire Line
-	5900 1150 5900 1200
-Wire Wire Line
-	6600 2000 6100 2000
-Wire Wire Line
-	6100 2000 5400 2000
-Wire Wire Line
-	5400 2450 5400 2850
-Connection ~ 5900 2850
-Wire Wire Line
-	5900 1700 5900 2300
-Wire Wire Line
-	5900 2300 5900 2350
-Wire Wire Line
-	5400 1200 5400 1150
-Wire Wire Line
-	4850 1150 4850 1200
-Wire Wire Line
-	5400 1700 5400 2000
-Wire Wire Line
-	5400 2000 5400 2050
-Connection ~ 5400 2000
-Connection ~ 5400 1150
-Wire Wire Line
-	4550 2000 4450 2000
-Wire Wire Line
-	5600 2550 4450 2550
-Wire Wire Line
-	3950 2250 3100 2250
-Wire Wire Line
-	8950 1800 8000 1800
-Wire Wire Line
-	8000 2000 8950 2000
-Wire Wire Line
-	8950 3500 6100 3500
-Wire Wire Line
-	1350 3850 1500 3850
-Wire Wire Line
-	1500 3850 1500 3950
-Wire Wire Line
-	6950 4750 7550 4750
 $Comp
 L R R?
@@
 IOIO_PIN1
 Text Label 8450 3500 0    60   ~ 0
-IOIO_PIN18
+IOIO_PIN14
 Text Label 8450 2100 0    60   ~ 0
 IOIO_PIN10

Commit message: Changes after opening in KiCad 0.201505041002+5641~23~ubunto14.04.1-product
I previously used kicad 0.20131208+bzr4024-1ubuntu2. Some other changes
might also not have been committed before.
Parts:
- added P?: CONN_8, symbol CONN_8
Changed lines of the file:
@@
-EESchema Schematic File Version 2  date Fri 14 Jun 2013 12:48:07 PM CEST
+EESchema Schematic File Version 2
 LIBS:power
 LIBS:device
@@
 LIBS:valves
 LIBS:ioio-adapter-cache
-EELAYER 25  0
+EELAYER 27 0
 EELAYER END
-$Descr A4 11700 8267
+$Descr A4 11693 8268
 encoding utf-8
 Sheet 1 1
 Title ""
-Date "14 jun 2013"
+Date "9 oct 2014"
 Rev ""
 Comp ""
@@
 F 0 "R?" V 6780 4750 50  0000 C CNN
 F 1 "100k" V 6700 4750 50  0000 C CNN
+F 2 "" H 6700 4750 60  0001 C CNN
+F 3 "" H 6700 4750 60  0001 C CNN
 	1    6700 4750
 	0    -1   -1   0
@@
 F 0 "#PWR?" H 1500 3590 20  0001 C CNN
 F 1 "+5V" H 1500 3590 30  0000 C CNN
+F 2 "" H 1500 3500 60  0001 C CNN
+F 3 "" H 1500 3500 60  0001 C CNN
 	1    1500 3500
 	1    0    0    -1
@@
 F 0 "#PWR?" H 1500 3950 30  0001 C CNN
 F 1 "GND" H 1500 3880 30  0001 C CNN
+F 2 "" H 1500 3950 60  0001 C CNN
+F 3 "" H 1500 3950 60  0001 C CNN
 	1    1500 3950
 	1    0    0    -1
@@
 F 0 "P?" V 950 3750 40  0000 C CNN
 F 1 "CONN_2" V 1050 3750 40  0000 C CNN
+F 2 "" H 1000 3750 60  0001 C CNN
+F 3 "" H 1000 3750 60  0001 C CNN
 	1    1000 3750
 	-1   0    0    1
@@
 F 0 "R?" V 4280 2550 50  0000 C CNN
 F 1 "5k" V 4200 2550 50  0000 C CNN
+F 2 "" H 4200 2550 60  0001 C CNN
+F 3 "" H 4200 2550 60  0001 C CNN
 	1    4200 2550
 	0    1    1    0
@@
 F 0 "R?" V 4280 2250 50  0000 C CNN
 F 1 "5k" V 4200 2250 50  0000 C CNN
+F 2 "" H 4200 2250 60  0001 C CNN
+F 3 "" H 4200 2250 60  0001 C CNN
 	1    4200 2250
 	0    1    1    0
@@
 F 0 "R?" V 4930 1450 50  0000 C CNN
 F 1 "10k" V 4850 1450 50  0000 C CNN
+F 2 "" H 4850 1450 60  0001 C CNN
+F 3 "" H 4850 1450 60  0001 C CNN
 	1    4850 1450
 	-1   0    0    1
@@
 F 0 "R?" V 5480 1450 50  0000 C CNN
 F 1 "10k" V 5400 1450 50  0000 C CNN
+F 2 "" H 5400 1450 60  0001 C CNN
+F 3 "" H 5400 1450 60  0001 C CNN
 	1    5400 1450
 	-1   0    0    1
@@
 F 0 "R?" V 5980 1450 50  0000 C CNN
 F 1 "10k" V 5900 1450 50  0000 C CNN
+F 2 "" H 5900 1450 60  0001 C CNN
+F 3 "" H 5900 1450 60  0001 C CNN
 	1    5900 1450
 	-1   0    0    1
@@
 F 0 "#PWR?" H 6400 3250 30  0001 C CNN
 F 1 "GND" H 6400 3180 30  0001 C CNN
+F 2 "" H 6400 3250 60  0001 C CNN
+F 3 "" H 6400 3250 60  0001 C CNN
 	1    6400 3250
 	1    0    0    -1
@@
 F 0 "#PWR?" H 6400 1140 20  0001 C CNN
 F 1 "+5V" H 6400 1140 30  0000 C CNN
+F 2 "" H 6400 1050 60  0001 C CNN
+F 3 "" H 6400 1050 60  0001 C CNN
 	1    6400 1050
 	1    0    0    -1
@@
 F 0 "R?" V 4280 2000 50  0000 C CNN
 F 1 "5k" V 4200 2000 50  0000 C CNN
+F 2 "" H 4200 2000 60  0001 C CNN
+F 3 "" H 4200 2000 60  0001 C CNN
 	1    4200 2000
 	0    1    1    0
@@
 F 0 "Q?" H 5300 2100 50  0000 R CNN
 F 1 "BC547" H 5300 2400 50  0000 R CNN
+F 2 "" H 5300 2250 60  0001 C CNN
+F 3 "" H 5300 2250 60  0001 C CNN
 	1    5300 2250
 	1    0    0    -1
@@
 F 0 "Q?" H 4750 1850 50  0000 R CNN
 F 1 "BC547" H 4750 2150 50  0000 R CNN
+F 2 "" H 4750 2000 60  0001 C CNN
+F 3 "" H 4750 2000 60  0001 C CNN
 	1    4750 2000
 	1    0    0    -1
@@
 F 0 "Q?" H 5800 2400 50  0000 R CNN
 F 1 "BC547" H 5800 2700 50  0000 R CNN
+F 2 "" H 5800 2550 60  0001 C CNN
+F 3 "" H 5800 2550 60  0001 C CNN
 	1    5800 2550
 	1    0    0    -1
@@
 F 0 "U?" H 7450 2850 70  0000 C CNN
 F 1 "74HC595" H 7300 1650 70  0000 C CNN
+F 2 "" H 7300 2250 60  0001 C CNN
+F 3 "" H 7300 2250 60  0001 C CNN
 	1    7300 2250
 	1    0    0    -1
@@
 F 0 "#PWR?" H 1500 2900 30  0001 C CNN
 F 1 "GND" H 1500 2830 30  0001 C CNN
+F 2 "" H 1500 2900 60  0001 C CNN
+F 3 "" H 1500 2900 60  0001 C CNN
 	1    1500 2900
 	1    0    0    -1
@@
 F 0 "K?" V 950 2600 50  0000 C CNN
 F 1 "CONN_3" V 1050 2600 40  0000 C CNN
+F 2 "" H 1000 2600 60  0001 C CNN
+F 3 "" H 1000 2600 60  0001 C CNN
 	1    1000 2600
 	-1   0    0    1
@@
 F 0 "#PWR?" H 1500 840 20  0001 C CNN
 F 1 "+5V" H 1500 840 30  0000 C CNN
+F 2 "" H 1500 750 60  0001 C CNN
+F 3 "" H 1500 750 60  0001 C CNN
 	1    1500 750
 	1    0    0    -1
@@
 F 0 "#PWR?" H 1500 1950 30  0001 C CNN
 F 1 "GND" H 1500 1880 30  0001 C CNN
+F 2 "" H 1500 1950 60  0001 C CNN
+F 3 "" H 1500 1950 60  0001 C CNN
 	1    1500 1950
 	1    0    0    -1
@@
 F 0 "J?" H 1000 1900 70  0000 C CNN
 F 1 "SIL10" V 1020 1300 70  0000 C CNN
+F 2 "" H 1000 1300 60  0001 C CNN
+F 3 "" H 1000 1300 60  0001 C CNN
 	1    1000 1300
 	-1   0    0    1
@@
 F 0 "R?" V 5680 5500 50  0000 C CNN
 F 1 "5k" V 5600 5500 50  0000 C CNN
+F 2 "" H 5600 5500 60  0001 C CNN
+F 3 "" H 5600 5500 60  0001 C CNN
 	1    5600 5500
 	0    1    1    0
@@
 F 0 "R?" V 6330 4400 50  0000 C CNN
 F 1 "100k" V 6250 4400 50  0000 C CNN
+F 2 "" H 6250 4400 60  0001 C CNN
+F 3 "" H 6250 4400 60  0001 C CNN
 	1    6250 4400
 	-1   0    0    1
@@
 F 0 "R?" V 5680 5000 50  0000 C CNN
 F 1 "5k" V 5600 5000 50  0000 C CNN
+F 2 "" H 5600 5000 60  0001 C CNN
+F 3 "" H 5600 5000 60  0001 C CNN
 	1    5600 5000
 	0    1    1    0
@@
 F 0 "#PWR?" H 6250 4060 30  0001 C CNN
 F 1 "+3.3V" H 6250 4210 30  0000 C CNN
+F 2 "" H 6250 4100 60  0001 C CNN
+F 3 "" H 6250 4100 60  0001 C CNN
 	1    6250 4100
 	1    0    0    -1
@@
 F 0 "#PWR?" H 6250 5850 30  0001 C CNN
 F 1 "GND" H 6250 5780 30  0001 C CNN
+F 2 "" H 6250 5850 60  0001 C CNN
+F 3 "" H 6250 5850 60  0001 C CNN
 	1    6250 5850
 	1    0    0    -1
@@
 F 0 "Q?" H 6150 5350 50  0000 R CNN
 F 1 "BC547" H 6150 5650 50  0000 R CNN
+F 2 "" H 6150 5500 60  0001 C CNN
+F 3 "" H 6150 5500 60  0001 C CNN
 	1    6150 5500
 	1    0    0    -1
@@
 F 0 "Q?" H 6150 4850 50  0000 R CNN
 F 1 "BC547" H 6150 5150 50  0000 R CNN
+F 2 "" H 6150 5000 60  0001 C CNN
+F 3 "" H 6150 5000 60  0001 C CNN
 	1    6150 5000
 	1    0    0    -1
 $EndComp
+$Comp
+L CONN_8 P?
+U 1 1 54366C7D
+P 1200 5600
+F 0 "P?" V 1150 5600 60  0000 C CNN
+F 1 "CONN_8" V 1250 5600 60  0000 C CNN
+F 2 "" H 1200 5600 60  0000 C CNN
+F 3 "" H 1200 5600 60  0000 C CNN
+	1    1200 5600
+	-1   0    0    1
+$EndComp
 $EndSCHEMATC
